File: thick_.sch (EAGLE design)
At the start: 37 parts, among them J4 F1003WR-S-06PT, Q1 SI2319DDS-T1-GE3, U1 ATTINY85-20SU, U2 TSR_0.5-2450

Commit message: rev 2
new pcb design with gerbers
Parts:
- removed C10: 4.7uF, resistor:C-EUC1206
- removed C11, C12: 0.1uF, resistor:C-EUC0603
- removed C9: 100uF, resistor:CPOL-EUE3.5-8
- removed D5, D6: 0.5A/40V/420mV, SparkFun-DiscreteSemi:DIODE-SCHOTTKY-PMEG4005EJ
- removed LED2: (no value), adafruit:LEDCHIPLED_0805
- removed R6: 10K, resistor:R-EU_R0603
- removed S1, S2: (no value), SparkFun-Switches:MOMENTARY-SWITCH-SPST-2-SMD-4.6X2.8MM
- D3: value tvs -> TVS; device SparkFun-DiscreteSemi:DIODE-SCHOTTKY-PMEG4005EJ -> diode:DIODE-DO214AC
- J1: value (none) -> 43045-0400; device SparkFun-Connectors:CONN_03LONGPADS -> 43045-0400:43045-0400
Connections:
- removed net N$4: LED2.A, R6.2
- removed net N$5: D6.A, J4.2
- removed net N$6: D3.C, D5.C, R2.1
- net !RESET: no longer C11.1, S1.1, S1.2
- net 5V: now also J4.2; no longer C10.1, D6.C, R1.1
- net AIN: now also U1.PB4; no longer U1.PB3
- net GND: now also J1.3; no longer C10.2, C11.2, C12.2, C9.-, J1.2, LED2.C, S1.3, S1.4, S2.3, S2.4
- net IGNITION: no longer R6.1
- net IGN_EN: now also U1.PB3; no longer U1.PB4
- net MOSI: now also D1.DI; no longer C12.1, S2.1, S2.2
- net SCK: no longer D1.DI
- net SIGNAL: now also D3.C, R2.1; no longer D5.A
- net VCC: now also J1.4; no longer J1.3
- net VDD: now also R1.1; no longer C9.+
Other:
- note removed: "RGA101M1HBK-0811G"
- moved on the sheet: C6, C7, C8, L1, U2
